Commit message: CLIK, nodes, msg (error catkin_make)

File: kuka_iiwa_14_prismatic_gripper/ros/iiwa.urdf (robot description, URDF)
Before this commit: robot iiwa14_gripper::iiwa14, 13 links, 12 joints
Links:
- removed link base_link_link
- removed link gripper_left_link
- removed link gripper_right_link
- removed link iiwa_link_ee
- removed link world
Joints:
- removed joint base_link_joint
- removed joint gripper_left_joint
- removed joint gripper_right_joint
- removed joint iiwa_joint_ee
- removed joint world_iiwa_joint
